Commit message: multiple drone controls were performed.

File: urdf/quad_cad.urdf (robot description, URDF)
Before this commit: robot quadcopter, 1 links, 0 joints
Links:
- link base_link: geometry collision mesh filename=package://multi_quadcopter_control/meshes/quad_model_v3.dae scale=0.008 0.008 0.008; visual mesh filename=package://multi_quadcopter_control/meshes/quad_model_v3.dae scale=0.008 0.008 0.008
