Commit message: scripts have been arranged.

File: urdf/quad_model_v2.urdf (robot description, URDF)
Before this commit: robot quadcopter, 1 links, 0 joints
Links:
- link base_link: geometry collision mesh filename=package://multi_quadcopter_control/meshes/quad_model_v4.dae scale=0.0018 0.0018 0.0018; visual mesh filename=package://multi_quadcopter_control/meshes/quad_model_v4.dae scale=0.0018 0.0018 0.0018
