Commit message: source code has been edited.

File: urdf/quad_model_v1.urdf (robot description, URDF)
Before this commit: robot quadcopter, 1 links, 0 joints
Links:
- link base_link: geometry collision mesh filename=package://multi_quadcopter_control/meshes/quad_model_v1.dae scale=0.005 0.005 0.005; visual mesh filename=package://multi_quadcopter_control/meshes/quad_model_v1.dae scale=0.005 0.005 0.005

File: urdf/quad_model_v2.urdf (robot description, URDF)
Before this commit: robot quadcopter, 1 links, 0 joints
Links:
- link base_link: geometry collision mesh filename=package://multi_quadcopter_control/meshes/quad_model_v2.dae scale=0.005 0.005 0.005; visual mesh filename=package://multi_quadcopter_control/meshes/quad_model_v2.dae scale=0.005 0.005 0.005

File: urdf/quad_model_v3.urdf (robot description, URDF)
Before this commit: robot quadcopter, 1 links, 0 joints
Links:
- link base_link: geometry collision mesh filename=package://multi_quadcopter_control/meshes/quad_model_v3.dae scale=0.005 0.005 0.005; visual mesh filename=package://multi_quadcopter_control/meshes/quad_model_v3.dae scale=0.005 0.005 0.005

Commit message: relative positions have been obtained.

File: urdf/quad_model_v1.urdf (robot description, URDF)
Before this commit: robot quadcopter, 1 links, 0 joints
Links:
- link base_link: geometry collision mesh filename=package://multi_quadcopter_control/meshes/quad_model_v1.dae scale=0.0018 0.0018 0.0018; visual mesh filename=package://multi_quadcopter_control/meshes/quad_model_v1.dae scale=0.0018 0.0018 0.0018

Commit message: file organization

File: urdf/quad_model_v1.urdf (robot description, URDF)
Before this commit: robot quadcopter, 1 links, 0 joints
Links:
- link base_link: geometry collision mesh filename=package://multi_quadcopter_control/meshes/quad_model_v1.dae scale=0.0010 0.0010 0.0010; visual mesh filename=package://multi_quadcopter_control/meshes/quad_model_v1.dae scale=0.0010 0.0010 0.0010

File: urdf/quad_model_v2.urdf (robot description, URDF)
Before this commit: robot quadcopter, 1 links, 0 joints
Links:
- link base_link: geometry collision mesh filename=package://multi_quadcopter_control/meshes/quad_model_v4.dae scale=0.0014 0.0014 0.0014; visual mesh filename=package://multi_quadcopter_control/meshes/quad_model_v4.dae scale=0.0014 0.0014 0.0014
